File: rtcl-p25k-usb3/rtcl-p25k-usb3.kicad_sch (KiCad schematic)
At the start: 6 parts, among them J1 USB3_B_Micro, U1 FT601Q, U2 TPD4E05U06DQA, U3 USBLC6-2P6

Commit message: Refactor code structure for improved readability and maintainability
Parts:
- added C3, C4: 18pF, symbol Device:C
- added C5, C6: 4.7uF, symbol Device:C
- added D1: PTVS5V0Z1USKP, Diode_SMD:Nexperia_DSN1608-2_1.6x0.8mm, symbol Diode:PTVS5V0Z1USKP
- added R1: 1.6k_1%, symbol Device:R
- added Y1: 30MHz, symbol Device:Crystal
Connections:
- net GND: now also U2.3 (GND), U2.8 (GND), C3.1, C4.1, C5.1, C6.1, D1.2 (A), R1.2
- net USB_SSRXM: now also U1.34 (RIDN), U2.2 (D1-)
- net USB_SSRXP: now also U1.35 (RIDP), U2.1 (D1+)
- net USB_SSTXM: now also C1.1, U2.5 (D2-)
- net USB_SSTXP: now also C2.1, U2.4 (D2+)
- net VBUS: now also C6.2, D1.1 (K)
- net FT601_TODP: now reaches C2.2, U1.32 (TODP)
- net at U1.2 (AVDD): now also U1.3 (VD10), U1.30 (VD10), U1.33 (VD10), U1.39 (DV10), U1.48 (VD10), C5.2
- net at U1.21 (XI): now also C3.2, Y1.1
- net at U1.22 (XO): now also C4.2, Y1.2
- net at U1.27 (RREF): now also R1.1
Other:
- moved on the sheet: U2, U3

Commit message: wip
Parts:
- added C68: <DNP>_C, symbol Device:C
- added C69: 47uF, symbol Device:C
- added C70: 4.7uF, symbol Device:C
- added C77, C78, C79: 4.7uF, Capacitor_SMD:C_0402_1005Metric, symbol Device:C_Small
- added J10, J11, J12: SSQ-106-02-F-D-RA, mipi_spartan7:PH_02x06_2.54mm, symbol Connector_Generic:Conn_02x06_Odd_Even
- added J2, J3: BTB-DF40C-60DS-0.4V(51), symbol Connector_Generic:Conn_02x30_Odd_Even
- added J7: RASPPICAM22, RASPPICAM22, symbol rtcl-xcaup-usb3:RASPPICAM22
- added R56: 1k, symbol Device:R
- added R57, R58: 2.2k, symbol Device:R
- added U12: TPS22917DBV, Package_TO_SOT_SMD:SOT-23-6, symbol Power_Management:TPS22917DBV
Connections:
- net GND: now also C69.2, C70.2, C77.2, C78.2, C79.2, J10.10 (Pin_10), J10.9 (Pin_9), J11.10 (Pin_10), J11.9 (Pin_9), J12.10 (Pin_10), J12.9 (Pin_9), J3.1 (Pin_1), J3.19 (Pin_19), J3.29 (Pin_29), J3.35 (Pin_35), J3.41 (Pin_41), J3.47 (Pin_47), J3.53 (Pin_53), J3.59 (Pin_59), J7.1 (GND), J7.10 (GND), J7.13 (GND), J7.16 (GND), J7.19 (GND), J7.4 (GND), J7.7 (GND), U12.2 (GND)
- new net: R56.1, U12.5 (QOD)
- new net: C70.1, J7.22 (3V3), R56.2, U12.6 (VOUT)
- new net: C68.2, U12.4 (CT)
- new net +1V8: J3.38 (Pin_38), J3.40 (Pin_40)
- new net +2V5: J3.42 (Pin_42), J3.44 (Pin_44)
- new net +3V3: J3.46 (Pin_46), J3.48 (Pin_48), J3.50 (Pin_50)
- new net A1_IOB24B_40P: J3.11 (Pin_11)
- new net A2_JTAG_TDO: J3.25 (Pin_25)
- new net A3_JTAG_TDI: J3.27 (Pin_27)
- new net B1_JTAG_TMS: J3.23 (Pin_23)
- new net B2_IOB4A_40P: J3.3 (Pin_3)
- new net C1_JTAG_TCK: J3.21 (Pin_21)
- new net C2_IOB4B_40P: J3.5 (Pin_5)
- new net D1_IOB14B_40P: J3.17 (Pin_17)
- new net D8_RECONFIG: J3.13 (Pin_13)
- new net E1_IOB12B_40P: J3.15 (Pin_15)
- new net F1_IOB26B_40P: J3.9 (Pin_9)
- new net F2_IOB26A_40P: J3.7 (Pin_7)
- new net G1_IOR24B_40P: J3.20 (Pin_20)
- new net G2_IOR24A_40P: J3.18 (Pin_18)
- new net J4_IOR22A_40P: J3.14 (Pin_14)
- new net K1_IOR20A_40P: J3.10 (Pin_10)
- new net K2_IOR20B_40P: J3.12 (Pin_12)
- new net K4_IOR22B_40P: J3.16 (Pin_16)
- new net L1_IOR18B_40P: J3.8 (Pin_8)
- new net L2_IOR18A_40P: J3.6 (Pin_6)
- new net L3_IOR31B_40P: J3.24 (Pin_24)
- new net L4_IOR31A_40P: J3.22 (Pin_22)
- new net M0_CK_N: J3.45 (Pin_45), J7.8 (CN)
- new net M0_CK_P: J3.43 (Pin_43), J7.9 (CP)
- new net M0_D0_N: J3.57 (Pin_57), J7.2 (DN0)
- new net M0_D0_P: J3.55 (Pin_55), J7.3 (DP0)
- new net M0_D1_N: J3.51 (Pin_51), J7.5 (DN1)
- new net M0_D1_P: J3.49 (Pin_49), J7.6 (DP1)
- new net M0_D2_N: J3.39 (Pin_39), J7.11 (DN2)
- new net M0_D2_P: J3.37 (Pin_37), J7.12 (DP2)
- new net M0_D3_N: J3.33 (Pin_33), J7.14 (DN3)
- new net M0_D3_P: J3.31 (Pin_31), J7.15 (DP3)
- new net MIPI3_GPIO0: J7.17 (GPIO0)
- new net MIPI3_GPIO1: J7.18 (GPIO1)
- new net MIPI3_PWR_ON: U12.3 (ON)
- new net MIPI3_SCK: J7.20 (SCL), R57.2
- new net MIPI3_SDA: J7.21 (SDA), R58.2
- new net PMOD_A0: J10.1 (Pin_1)
- new net PMOD_A1: J10.3 (Pin_3)
- new net PMOD_A2: J10.5 (Pin_5)
- new net PMOD_A3: J10.7 (Pin_7)
- new net PMOD_A4: J10.2 (Pin_2)
- new net PMOD_A5: J10.4 (Pin_4)
- new net PMOD_A6: J10.6 (Pin_6)
- new net PMOD_A7: J10.8 (Pin_8)
- new net PMOD_B0: J11.1 (Pin_1)
- new net PMOD_B1: J11.3 (Pin_3)
- new net PMOD_B2: J11.5 (Pin_5)
- new net PMOD_B3: J11.7 (Pin_7)
- new net PMOD_B4: J11.2 (Pin_2)
- new net PMOD_B5: J11.4 (Pin_4)
- new net PMOD_B6: J11.6 (Pin_6)
- new net PMOD_B7: J11.8 (Pin_8)
- new net PMOD_C0: J12.1 (Pin_1)
- new net PMOD_C1: J12.3 (Pin_3)
- new net PMOD_C2: J12.5 (Pin_5)
- new net PMOD_C3: J12.7 (Pin_7)
- new net PMOD_C4: J12.2 (Pin_2)
- new net PMOD_C5: J12.4 (Pin_4)
- new net PMOD_C6: J12.6 (Pin_6)
- new net PMOD_C7: J12.8 (Pin_8)
- new net VCCIO2_3: J3.2 (Pin_2), J3.4 (Pin_4)
- new net VCCIO33: C68.1, C69.1, C77.1, C78.1, C79.1, J10.11 (Pin_11), J10.12 (Pin_12), J11.11 (Pin_11), J11.12 (Pin_12), J12.11 (Pin_11), J12.12 (Pin_12), R57.1, R58.1, U12.1 (VIN)
Other:
- note added: "BANK10"
- note added: "BANK5"
- note added: "GCLK"
- note added: "MIPI"

Commit message: WIP
Connections:
- net VBUS is gone; now on net +5V: C6.2, D1.1 (K), J1.1 (VBUS), U3.5 (VBUS)
- net GND: now also J2.1 (Pin_1), J2.15 (Pin_15), J2.2 (Pin_2), J2.27 (Pin_27), J2.28 (Pin_28), J2.45 (Pin_45), J2.50 (Pin_50), J2.59 (Pin_59), J2.60 (Pin_60)
- net K5_IOT63B: now reaches J2.10 (Pin_10)
- net F7_IOT58A_40P: now reaches J2.11 (Pin_11)
- net H8_IOT66A: now reaches J2.12 (Pin_12)
- net F6_IOT58B_40P: now reaches J2.13 (Pin_13)
- net H7_IOT66B: now reaches J2.14 (Pin_14)
- net G7_IOT68A: now reaches J2.16 (Pin_16)
- net E8_READY: now reaches J2.17 (Pin_17)
- net G7_IOT68B: now reaches J2.18 (Pin_18)
- net B3_IOB56A_UART_RX: now reaches J2.19 (Pin_19)
- net C3_IOB56B_UART_TX: now reaches J2.21 (Pin_21)
- net E3_IOB60A_40P: now reaches J2.23 (Pin_23)
- net D7_DONE: now reaches J2.25 (Pin_25)
- net VCCIO6_7: now reaches J2.29 (Pin_29)
- net VCCIO6_7: now also J2.31 (Pin_31)
- net L9_IOT31A_40P: now reaches J2.3 (Pin_3)
- net J11_IOT1A_40P: now reaches J2.33 (Pin_33)
- net J10_IOT1B_40P: now reaches J2.35 (Pin_35)
- net H11_IOT3A_S1: now reaches J2.37 (Pin_37)
- net H10_IOT3B_S2: now reaches J2.39 (Pin_39)
- net H5_IOT61A: now reaches J2.4 (Pin_4)
- net G11_IOT7A: now reaches J2.41 (Pin_41)
- net G10_IOT7B: now reaches J2.43 (Pin_43)
- net D11_IOL9A: now reaches J2.47 (Pin_47)
- net D10_IOL9B: now reaches J2.49 (Pin_49)
- net K9_IOT31B_40P: now reaches J2.5 (Pin_5)
- net C11_IOL5A: now reaches J2.51 (Pin_51)
- net C10_IOL5B: now reaches J2.53 (Pin_53)
- net B11_IOL12A: now reaches J2.55 (Pin_55)
- net B10_IOL12B: now reaches J2.57 (Pin_57)
- net J5_IOT61B: now reaches J2.6 (Pin_6)
- net J8_IOT56A_40P: now reaches J2.7 (Pin_7)
- net L5_IOT63A: now reaches J2.8 (Pin_8)
- net K8_IOT56B_40P: now reaches J2.9 (Pin_9)
- net J1_IOR33A_40P: now reaches J3.26 (Pin_26)
- net J2_IOR33B_40P: now reaches J3.28 (Pin_28)
- net G4_IOB89A_40P: now reaches J3.30 (Pin_30)
- net H4_IOB89B_40P: now reaches J3.32 (Pin_32)
- net H1_IOB91A_40P: now reaches J3.34 (Pin_34)
- net H2_IOB91B_40P: now reaches J3.36 (Pin_36)
- net +5V: now reaches J3.52 (Pin_52)
- net +5V: now also J3.54 (Pin_54), J3.56 (Pin_56), J3.58 (Pin_58), J3.60 (Pin_60)
Other:
- note added: "BANK0"
- note added: "BANK2"
- note added: "BANK3"
- note added: "BANK4"
- note added: "BANK6"
- note added: "BANK7"
- note added: "RPLL"
- moved on the sheet: J2, J3

Commit message: WIP
Connections:
- net F5_IOT72A: now reaches J2.20 (Pin_20)
- net G5_IOT72B: now reaches J2.22 (Pin_22)
- net VCCIO0_1: now reaches J2.24 (Pin_24)
- net VCCIO0_1: now also J2.26 (Pin_26)
- net L6_IOT23A_USB_P: now reaches J2.30 (Pin_30)
- net K6_IOT23B_USB_N: now reaches J2.32 (Pin_32)
- net K7_IOT21A_40P: now reaches J2.34 (Pin_34)
- net J7_IOT21B_40P: now reaches J2.36 (Pin_36)
- net L7_IOT19A_40P: now reaches J2.38 (Pin_38)
- net L8_IOT19B_40P: now reaches J2.40 (Pin_40)
- net L10_IOT15A_40P: now reaches J2.42 (Pin_42)
- net K10_IOT15B_40P: now reaches J2.44 (Pin_44)
- net K11_IOT11A: now reaches J2.46 (Pin_46)
- net L11_IOT11B: now reaches J2.48 (Pin_48)
- net E11_IOL3A: now reaches J2.52 (Pin_52)
- net E10_IOL3B: now reaches J2.54 (Pin_54)
- net A11_IOL14A: now reaches J2.56 (Pin_56)
- net A10_IOL14B: now reaches J2.58 (Pin_58)
Other:
- moved on the sheet: J2

Commit message: Refactor code structure for improved readability and maintainability
Parts:
- added C10, C11, C7, C8, C9: 0.1uF, symbol Device:C
- added C12, C13, C14: 4.7uF, symbol Device:C
- added J5: JTAG, symbol Connector_Generic:Conn_01x06
- added R10, R11, R12, R13, R14, R15, R16, R17, R18, R19, R20, R21, R22, R23, R24, R25, R26, R27, R28, R29, R30, R31, R32, R33, R34, R35, R36, R37, R38, R39, R4, R40, R41, R42, R43, R44, R45, R46, R47, R48, R5, R6, R7, R8, R9: 22, symbol Device:R
- added R2: 4.7k, symbol Device:R
- added R3: 10k, symbol Device:R
- added R49, R50, R51, R52: 0, symbol Device:R
- added R53, R54: <DNP>_R, symbol Device:R
- renumbered J7 to J2, J2 to J3, J3 to J4
Connections:
- net +1V8: now also R54.1
- net +2V5: now also R53.1
- net +3V3: now also U1.20 (VCC33), U1.24 (VCC33), U1.28 (VDDA), U1.38 (VCC33), C8.2, C9.2, J5.6 (Pin_6), R52.1
- net +5V: now also U1.37 (VBUS), C10.2
- net A2_JTAG_TDO: now also J5.3 (Pin_3)
- net A3_JTAG_TDI: now also J5.2 (Pin_2)
- net B1_JTAG_TMS: now also J5.1 (Pin_1)
- net C1_JTAG_TCK: now also J5.4 (Pin_4)
- net GND: now also U1.1 (GND), U1.26 (GND), U1.29 (GND), U1.36 (GND), U1.77 (GND), C10.1, C11.1, C12.1, C13.1, C14.1, C7.1, C8.1, C9.1, J5.5 (Pin_5)
- net VCCIO0_1: now also C12.2, R49.2
- net VCCIO2_3: now also C13.2, R50.2
- net VCCIO6_7: now also C14.2, R51.2
- net FT601_CLK: now reaches U1.10 (~{SIWU})
- net FT601_CLK: now also U1.58 (CLK), R4.1, R43.1
- net FT601_WR: now reaches U1.11 (~{WR})
- net FT601_WR: now also R44.1
- net FT601_RD: now reaches U1.12 (~{RD})
- net FT601_RD: now also R45.1
- net FT601_OE: now reaches U1.13 (~{OE})
- net FT601_OE: now also R46.1
- net VCC: now reaches U1.14 (VCCIO), U1.49 (VCCIO), U1.59 (VCCIO), U1.68 (VCCIO)
- net VCC: now also C7.2, R2.1, R3.2, R49.1, R50.1, R51.1, R52.2, R53.2, R54.2
- net FT601_RESET: now reaches U1.15 (~{RESET})
- net FT601_RESET: now also C11.2, R3.1
- net at U1.16 (~{WAKEUP}): now also R2.2
- net FT601_GPIO0: now reaches U1.17 (GPIO0)
- net FT601_GPIO0: now also R47.1
- net FT601_GPIO1: now reaches U1.18 (GPIO1)
- net FT601_GPIO1: now also R48.1
- net FT601_BE0: now reaches U1.4 (BE_0)
- net FT601_BE0: now also R39.1
- net FT601_D0: now reaches U1.40 (DATA_0)
- net FT601_D0: now also R7.1
- net FT601_D1: now reaches U1.41 (DATA_1)
- net FT601_D1: now also R8.1
- net FT601_D2: now reaches U1.42 (DATA_2)
- net FT601_D2: now also R9.1
- net FT601_D3: now reaches U1.43 (DATA_3)
- net FT601_D3: now also R10.1
- net FT601_D4: now reaches U1.44 (DATA_4)
- net FT601_D4: now also R11.1
- net FT601_D5: now reaches U1.45 (DATA_5)
- net FT601_D5: now also R12.1
- net FT601_D6: now reaches U1.46 (DATA_6)
- net FT601_D6: now also R13.1
- net FT601_D7: now reaches U1.47 (DATA_7)
- net FT601_D7: now also R14.1
- net FT601_BE1: now reaches U1.5 (BE_1)
- net FT601_BE1: now also R40.1
- net FT601_D8: now reaches U1.50 (DATA_8)
- net FT601_D8: now also R15.1
- net FT601_D9: now reaches U1.51 (DATA_9)
- net FT601_D9: now also R16.1
- net FT601_D10: now reaches U1.52 (DATA_10)
- net FT601_D10: now also R17.1
- net FT601_D11: now reaches U1.53 (DATA_11)
- net FT601_D11: now also R18.1
- net FT601_D12: now reaches U1.54 (DATA_12)
- net FT601_D12: now also R19.1
- net FT601_D13: now reaches U1.55 (DATA_13)
- net FT601_D13: now also R20.1
- net FT601_D14: now reaches U1.56 (DATA_14)
- net FT601_D14: now also R21.1
- net FT601_D15: now reaches U1.57 (DATA_15)
- net FT601_D15: now also R22.1
- net FT601_BE2: now reaches U1.6 (BE_2)
- net FT601_BE2: now also R41.1
- net FT601_D16: now reaches U1.60 (DATA_16)
- net FT601_D16: now also U1.69 (DATA_24), R23.1, R31.1
- net FT601_D17: now reaches U1.61 (DATA_17)
- net FT601_D17: now also U1.70 (DATA_25), R24.1, R32.1
- net FT601_D18: now reaches U1.62 (DATA_18)
- net FT601_D18: now also U1.71 (DATA_26), R25.1, R33.1
- net FT601_D19: now reaches U1.63 (DATA_19)
- net FT601_D19: now also U1.72 (DATA_27), R26.1, R34.1
- net FT601_D20: now reaches U1.64 (DATA_20)
- net FT601_D20: now also U1.73 (DATA_28), R27.1, R35.1
- net FT601_D21: now reaches U1.65 (DATA_21)
- net FT601_D21: now also U1.74 (DATA_29), R28.1, R36.1
- net FT601_D22: now reaches U1.66 (DATA_22)
- net FT601_D22: now also U1.75 (DATA_30), R29.1, R37.1
- net FT601_D23: now reaches U1.67 (DATA_23)
- net FT601_D23: now also U1.76 (DATA_31), R30.1, R38.1
- net FT601_BE3: now reaches U1.7 (BE_3)
- net FT601_BE3: now also R42.1
- net FT601_TXE: now reaches U1.8 (~{TXE})
- net FT601_TXE: now also R5.1
- net FT601_RXF: now reaches U1.9 (~{RXF})
- net FT601_RXF: now also R6.1
- net A1_IOB24B_40P renamed A1_IOB24A_40P
Other:
- note added: "3.3V"
- moved on the sheet: C1, C2, C3, C4, C5, C6, C68, C69, C70, C77, C78, C79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

Commit message: WIP
Parts:
- removed C78, C79: 4.7uF, Capacitor_SMD:C_0402_1005Metric, symbol Device:C_Small
- removed J11, J12: SSQ-106-02-F-D-RA, mipi_spartan7:PH_02x06_2.54mm, symbol Connector_Generic:Conn_02x06_Odd_Even
- added L1: BLM18PG221SN1D, Inductor_SMD:L_0603_1608Metric, symbol Device:L
- added R55: 0, Resistor_SMD:R_0603_1608Metric, symbol Device:R
- C1, C10, C11, C2, C3, C4, C7, C8, C9: footprint (none) -> Capacitor_SMD:C_0402_1005Metric
- C12, C13, C14, C5, C6, C68, C70: footprint (none) -> Capacitor_SMD:C_0603_1608Metric
- C69: footprint (none) -> Capacitor_SMD:C_0805_2012Metric
- J5: footprint (none) -> Connector_PinHeader_2.54mm:PinHeader_1x08_P2.54mm_Vertical
- R1, R10, R11, R12, R13, R14, R15, R16, R17, R18, R19, R2, R20, R21, R22, R23, R24, R25, R26, R27, R28, R29, R3, R30, R31, R32, R33, R34, R35, R36, R37, R38, R39, R4, R40, R41, R42, R43, R44, R45, R46, R47, R48, R49, R5, R50, R51, R52, R53, R54, R56, R57, R58, R6, R7, R8, R9: footprint (none) -> Resistor_SMD:R_0603_1608Metric
Connections:
- net E3_IOB60A_40P is gone; now on net B3_IOB56A_UART_RX: J3.23 (Pin_23)
- net MIPI3_GPIO0 is gone; now on net B3_IOB56A_UART_RX: J2.17 (GPIO0)
- net MIPI3_GPIO1 is gone; now on net C3_IOB56B_UART_TX: J2.18 (GPIO1)
- net PMOD_A0 is gone; now on net B2_IOB4A_40P: J10.1 (Pin_1)
- net PMOD_A1 is gone; now on net C2_IOB4B_40P: J10.3 (Pin_3)
- net PMOD_A2 is gone; now on net F2_IOB26A_40P: J10.5 (Pin_5)
- net PMOD_A3 is gone; now on net F1_IOB26B_40P: J10.7 (Pin_7)
- net PMOD_A4 is gone; now on net A1_IOB24A_40P: J10.2 (Pin_2)
- net PMOD_A5 is gone; now on net D8_RECONFIG: J10.4 (Pin_4)
- net PMOD_A6 is gone; now on net E1_IOB12B_40P: J10.6 (Pin_6)
- net PMOD_A7 is gone; now on net D1_IOB14B_40P: J10.8 (Pin_8)
- net GND: now also L1.2, R55.2
- net at J1.8 (DRAIN): now also R55.1
- net at J1.SH (SHIELD): now also L1.1

Commit message: WIP
Parts:
- added RN1: R_Pack04, Resistor_SMD:R_Array_Convex_4x0603, symbol Device:R_Pack04
- L1: footprint Inductor_SMD:L_0603_1608Metric -> Resistor_SMD:R_0402_1005Metric
- R1, R10, R11, R12, R13, R14, R15, R16, R17, R18, R19, R2, R20, R21, R22, R23, R24, R25, R26, R27, R28, R29, R3, R30, R31, R32, R33, R34, R35, R36, R37, R38, R39, R4, R40, R41, R42, R43, R44, R45, R46, R47, R48, R49, R5, R50, R51, R52, R53, R54, R55, R56, R57, R58, R6, R7, R8, R9: footprint Resistor_SMD:R_0603_1608Metric -> Resistor_SMD:R_0402_1005Metric
Connections:
- net FT601_BE0: now also RN1.5 (R4.2); no longer R39.1
- net FT601_BE1: now also RN1.6 (R3.2); no longer R40.1
- net FT601_BE2: now also RN1.7 (R2.2); no longer R41.1
- net FT601_BE3: now also RN1.8 (R1.2); no longer R42.1
Other:
- moved on the sheet: R39, R40, R41, R42

Commit message: WIP
Parts:
- J3, J4: footprint (none) -> rtcl-p25k-usb3:CONN_DF40C-60DS_HIR
- renumbered Y1 to X1
Changed lines of the file:
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@@
 			)
 		)
-		(property "Footprint" ""
+		(property "Footprint" "rtcl-p25k-usb3:CONN_DF40C-60DS_HIR"
 			(at 248.92 71.12 0)
 			(hide yes)
@@
 			)
 		)
-		(property "Footprint" ""
+		(property "Footprint" "rtcl-p25k-usb3:CONN_DF40C-60DS_HIR"
 			(at 351.79 71.12 0)
 			(hide yes)
@@
 		(dnp no)
 		(fields_autoplaced yes)
-		(property "Reference" "Y1"
+		(property "Reference" "X1"
 			(at 102.87 262.8899 90)
 			(show_name no)
@@
 			(project "rtcl-p25k-usb3"
 				(path "/3111823c-3b86-4a35-a2d4-382a0824eec6"
-					(reference "Y1")
+					(reference "X1")
 					(unit 1)
 				)
