File: rtcl-tp25k-usb3/rtcl-tp25k-usb3.kicad_sch (KiCad schematic)
At the start: 65 parts, among them J1 ZX360D-B-10P(30), J10 SSQ-106-02-F-D-RA, J2 0525592253, J3 BTB-DF40C-60DS-0.4V(51), J4 DF40C-60DS-0.4V(51), J5 JTAG, U1 FT601Q, U12 TPS22917DBV, U2 TPD4E05U06DQA, U3 USBLC6-2P6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

Commit message: Update model paths in KiCad module files for consistency
- Changed model path for CONN10_ZX360D-B-10P30_HIR.kicad_mod to reflect the correct directory structure.
- Updated model path for CONN_DF40C-60DS_HIR.kicad_mod to point to the new location.
- Modified model path for CON_525592253_MOL.kicad_mod to ensure it aligns with the updated project directory.
Parts:
- J1: footprint rtcl-p25k-usb3:CONN10_ZX360D-B-10P30_HIR -> rtcl-tp25k-usb3:CONN10_ZX360D-B-10P30_HIR
- J10: footprint rtcl-p25k-usb3:PMOD_02x06_2.54mm -> rtcl-tp25k-usb3:PMOD_02x06_2.54mm
- J2: footprint rtcl-p25k-usb3:CON_525592253_MOL -> rtcl-tp25k-usb3:CON_525592253_MOL
- J3, J4: footprint rtcl-p25k-usb3:CONN_DF40C-60DS_HIR -> rtcl-tp25k-usb3:CONN_DF40C-60DS_HIR
- RN1, RN2, RN3, RN4, RN5, RN6, RN7, RN8, RN9: footprint rtcl-p25k-usb3:RES_YC104_YAG -> rtcl-tp25k-usb3:RES_YC104_YAG
- RN999, RN9998: footprint rtcl-p25k-usb3:RES_YC164_3P2X1P6_YAG -> rtcl-tp25k-usb3:RES_YC164_3P2X1P6_YAG
- U1: symbol rtcl-p25k-usb3:FT601Q -> rtcl-tp25k-usb3:FT601Q

Commit message: WIP
Parts:
- removed C68: <DNP>_C, Capacitor_SMD:C_0603_1608Metric, symbol Device:C
- removed C69: 47uF, Capacitor_SMD:C_0805_2012Metric, symbol Device:C
- removed C70: 4.7uF, Capacitor_SMD:C_0603_1608Metric, symbol Device:C
- removed R56: 1k, Resistor_SMD:R_0402_1005Metric, symbol Device:R
- removed RN999: YC164-JR-0722RL, rtcl-tp25k-usb3:RES_YC164_3P2X1P6_YAG, symbol Device:R_Pack04
- removed RN9998: YC124-JR-1322RL, rtcl-tp25k-usb3:RES_YC164_3P2X1P6_YAG, symbol Device:R_Pack04
- removed U12: TPS22917DBV, Package_TO_SOT_SMD:SOT-23-6, symbol Power_Management:TPS22917DBV
- added C71, C72: 4.7uF, Capacitor_SMD:C_0603_1608Metric, symbol Device:C
- added C73: 120pF, Capacitor_SMD:C_0603_1608Metric, symbol Device:C
- added L1: TFM201610ALM-R47MTAA, rtcl-p25k-usb3:INDC2016X100N, symbol Device:L
- added R60: 22.6k_1%, Resistor_SMD:R_0402_1005Metric, symbol Device:R
- added R61: 100k_1%, Resistor_SMD:R_0402_1005Metric, symbol Device:R
- added U4: TPS62826DMQR, rtcl-p25k-usb3:DMQ0006A, symbol rtcl-tp25k-usb3:TPS62826DMQR
- FB1: footprint (none) -> Inductor_SMD:L_0603_1608Metric
- J1: footprint rtcl-tp25k-usb3:CONN10_ZX360D-B-10P30_HIR -> rtcl-p25k-usb3:CONN10_ZX360D-B-10P30_HIR
- J10: footprint rtcl-tp25k-usb3:PMOD_02x06_2.54mm -> rtcl-p25k-usb3:PMOD_02x06_2.54mm
- J2: footprint rtcl-tp25k-usb3:CON_525592253_MOL -> rtcl-p25k-usb3:CON_525592253_MOL
- J3, J4: footprint rtcl-tp25k-usb3:CONN_DF40C-60DS_HIR -> rtcl-p25k-usb3:CONN_DF40C-60DS_HIR
- R52: value 0 -> 0_1608
- R53, R54: value <DNP>_R -> <DNP>_R_1608
- RN1, RN2, RN3, RN4, RN5, RN6, RN7, RN8, RN9: footprint rtcl-tp25k-usb3:RES_YC104_YAG -> rtcl-p25k-usb3:RES_YC104_YAG
- X1: value 30MHz -> ABM3-30.000MHZ-D2Y-T; LCSC (none) -> C5371650
Connections:
- net +1V8: now also R52.1; no longer R54.1
- net +3V3: now also R54.1; no longer R52.1
- net +5V: now also C71.1, U4.6 (VIN)
- net D8_RECONFIG: no longer J10.4 (Pin_4)
- net GND: now also C71.2, C72.2, R60.2, U4.4 (GND)
- net VCCIO33: no longer R57.1, R58.1
- net +3.3VP: now reaches J2.22 (3V3)
- net +3.3VP: now also R57.1, R58.1, C72.1, C73.1, L1.2, R61.1
- net USB_SSRXM renamed USB_SSRX_N
- net USB_SSRXP renamed USB_SSRX_P
- net USB_SSTXM renamed USB_SSTX_N
- net USB_SSTXP renamed USB_SSTX_P
- new net: C73.2, R60.1, R61.2, U4.3 (FB)
- new net: L1.1, U4.5 (SW)
- new net MIPI_PWR_EN: U4.1 (EN)
- new net PGOOD: U4.2 (PG)
- new net PMOD_A5: J10.4 (Pin_4)
Other:
- moved on the sheet: R52, R54

Commit message: WIP
Parts:
- removed X1: ABM3-30.000MHZ-D2Y-T, symbol Device:Crystal
- added X1: ABM8-30.000MHZ-D1X-T, rtcl-p25k-usb3:XTAL_ABM8-30.000MHz-D1X-T, symbol rtcl-tp25k-usb3:ABM8-30.000MHZ-D1X-T
- R52, R53, R54: footprint Resistor_SMD:R_0402_1005Metric -> Resistor_SMD:R_0603_1608Metric_Pad0.98x0.95mm_HandSolder
Connections:
- net GND: now also X1.2 (GND), X1.4 (GND)
- net at C3.2, U1.21 (XI): now also X1.3
- net at C4.2, U1.22 (XO): now also X1.1
Other:
- moved on the sheet: C3, C4

Commit message: WIP
Parts:
- added C74: 0.1uF, Capacitor_SMD:C_0402_1005Metric, symbol Device:C
- added R62: 200k, Resistor_SMD:R_0402_1005Metric, symbol Device:R
- added R63, R64: 2.2k, Resistor_SMD:R_0402_1005Metric, symbol Device:R
- added U5: PCA9306DC, Package_SO:VSSOP-8_2.3x2mm_P0.5mm, symbol Interface:PCA9306DC
- C73: footprint Capacitor_SMD:C_0603_1608Metric -> Capacitor_SMD:C_0402_1005Metric
- C77: footprint Capacitor_SMD:C_0402_1005Metric -> Capacitor_SMD:C_0603_1608Metric
Connections:
- net +3.3VP: now also R62.1, R63.1, R64.1
- net GND: now also C74.2, U5.1 (GND)
- net MIPI_SCL: now also U5.6 (SCL2)
- net MIPI_SDA: now also U5.5 (SDA2)
- net VCC: now also C74.1, U5.2 (VREF1)
- new net: R62.2, U5.7 (VREF2), U5.8 (EN)
- new net: R63.2, U5.3 (SCL1)
- new net: R64.2, U5.4 (SDA1)
Other:
- moved on the sheet: J2, R57, R58

Commit message: WIP
Parts:
- added C21, C22, C23, C24, C25: 0.1uF, Capacitor_SMD:C_0402_1005Metric, symbol Device:C
- added FB2: BLM18SG121TN1, Inductor_SMD:L_0603_1608Metric, symbol Device:FerriteBead
Connections:
- net +5V: now also C10.2, U1.37 (VBUS)
- net GND: now also C21.1, C22.1, C23.1, C24.1, C25.1
- net USB_SSRX_N: now also U2.7 (NC)
- net USB_SSRX_P: now also U2.6 (NC)
- net USB_SSTX_N: now also U2.10 (NC)
- net USB_SSTX_P: now also U2.9 (NC)
- net VBUS: no longer C10.2, U1.37 (VBUS)
- net at C5.2, U1.3 (VD10), U1.30 (VD10)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: now also C21.2, C22.2, C23.2, C24.2, FB2.2; no longer U1.2 (AVDD)
- net FT601_DM renamed FT601_D_N
- net FT601_DP renamed FT601_D_P
- net USB_DM renamed USB_D_N
- net USB_DP renamed USB_D_P
- new net: C25.2, FB2.1, U1.2 (AVDD)
Other:
- moved on the sheet: C5

Commit message: Refactor code structure for improved readability and maintainability
Connections:
- net B10_IOL12B: now also RN2.5 (R4.2)
- net B11_IOL12A: now also RN2.6 (R3.2)
- net C10_IOL5B: now also RN2.7 (R2.2)
- net C11_IOL5A: now also RN2.8 (R1.2)
- net D10_IOL9B: now also RN3.5 (R4.2)
- net D11_IOL9A: now also RN3.6 (R3.2)
- net F6_IOT58B_40P: now also RN5.5 (R4.2)
- net F7_IOT58A_40P: now also RN5.6 (R3.2)
- net FT601_D16: no longer RN8.4 (R4.1), U1.69 (DATA_24)
- net FT601_D17: no longer RN8.3 (R3.1), U1.70 (DATA_25)
- net FT601_D18: no longer RN8.2 (R2.1), U1.71 (DATA_26)
- net FT601_D19: no longer RN8.1 (R1.1), U1.72 (DATA_27)
- net FT601_D20: no longer RN9.4 (R4.1), U1.73 (DATA_28)
- net FT601_D21: no longer RN9.3 (R3.1), U1.74 (DATA_29)
- net FT601_D22: no longer RN9.2 (R2.1), U1.75 (DATA_30)
- net FT601_D23: no longer RN9.1 (R1.1), U1.76 (DATA_31)
- net G10_IOT7B: now also RN3.7 (R2.2)
- net G11_IOT7A: now also RN3.8 (R1.2)
- net G7_IOT68A: now also RN7.7 (R2.2)
- net G8_IOT68B: now also RN7.8 (R1.2)
- net H10_IOT3B_S2: now also RN4.5 (R4.2)
- net H11_IOT3A_S1: now also RN4.6 (R3.2)
- net H5_IOT61A: now also RN6.5 (R4.2)
- net H7_IOT66B: now also RN7.6 (R3.2)
- net H8_IOT66A: now also RN7.5 (R4.2)
- net J10_IOT1B_40P: now also RN4.7 (R2.2)
- net J11_IOT1A_40P: now also RN4.8 (R1.2)
- net J5_IOT61B: now also RN6.6 (R3.2)
- net J8_IOT56A_40P: now also R43.2
- net K5_IOT63B: now also RN6.8 (R1.2)
- net K8_IOT56B_40P: now also RN5.7 (R2.2)
- net K9_IOT31B_40P: now also RN5.8 (R1.2)
- net L5_IOT63A: now also RN6.7 (R2.2)
- net at C25.2, FB2.1: no longer U1.2 (AVDD)
- new net FT601_D24: RN8.4 (R4.1), U1.69 (DATA_24)
- new net FT601_D25: RN8.3 (R3.1), U1.70 (DATA_25)
- new net FT601_D26: RN8.2 (R2.1), U1.71 (DATA_26)
- new net FT601_D27: RN8.1 (R1.1), U1.72 (DATA_27)
- new net FT601_D28: RN9.4 (R4.1), U1.73 (DATA_28)
- new net FT601_D29: RN9.3 (R3.1), U1.74 (DATA_29)
- new net FT601_D30: RN9.2 (R2.1), U1.75 (DATA_30)
- new net FT601_D31: RN9.1 (R1.1), U1.76 (DATA_31)
Other:
- moved on the sheet: C12, C13, C14, C77, J10, J3, J4, J5, R49, R50, R51, R52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

Commit message: Refactor code structure for improved readability and maintainability
Connections:
- net G4_IOB89A_40P is gone; now on net FT601_RESET: J4.30 (Pin_30)
- net H4_IOB89B_40P is gone; now on net FT601_WAKEUP: J4.32 (Pin_32)
- net B10_IOL12B: no longer RN2.5 (R4.2)
- net B11_IOL12A: no longer RN2.6 (R3.2)
- net C10_IOL5B: no longer RN2.7 (R2.2)
- net C11_IOL5A: now also RN2.5 (R4.2); no longer RN2.8 (R1.2)
- net D10_IOL9B: now also RN2.6 (R3.2); no longer RN3.5 (R4.2)
- net D11_IOL9A: now also RN2.7 (R2.2); no longer RN3.6 (R3.2)
- net F5_IOT72A: now also RN7.7 (R2.2)
- net F6_IOT58B_40P: now also RN4.6 (R3.2); no longer RN5.5 (R4.2)
- net F7_IOT58A_40P: now also RN4.7 (R2.2); no longer RN5.6 (R3.2)
- net G10_IOT7B: now also RN2.8 (R1.2); no longer RN3.7 (R2.2)
- net G11_IOT7A: now also RN3.5 (R4.2); no longer RN3.8 (R1.2)
- net G5_IOT72B: now also RN7.8 (R1.2)
- net G7_IOT68A: now also RN7.5 (R4.2); no longer RN7.7 (R2.2)
- net G8_IOT68B: now also RN7.6 (R3.2); no longer RN7.8 (R1.2)
- net H10_IOT3B_S2: now also RN3.6 (R3.2); no longer RN4.5 (R4.2)
- net H11_IOT3A_S1: now also RN3.7 (R2.2); no longer RN4.6 (R3.2)
- net H1_IOB91A_40P: now also R46.2
- net H2_IOB91B_40P: now also R47.2
- net H5_IOT61A: now also RN5.8 (R1.2); no longer RN6.5 (R4.2)
- net H7_IOT66B: now also RN6.8 (R1.2); no longer RN7.6 (R3.2)
- net H8_IOT66A: now also RN6.7 (R2.2); no longer RN7.5 (R4.2)
- net J10_IOT1B_40P: now also RN3.8 (R1.2); no longer RN4.7 (R2.2)
- net J11_IOT1A_40P: now also RN4.5 (R4.2); no longer RN4.8 (R1.2)
- net J5_IOT61B: now also R43.2; no longer RN6.6 (R3.2)
- net J8_IOT56A_40P: now also RN5.5 (R4.2); no longer R43.2
- net K5_IOT63B: now also RN6.6 (R3.2); no longer RN6.8 (R1.2)
- net K8_IOT56B_40P: now also RN4.8 (R1.2); no longer RN5.7 (R2.2)
- net K9_IOT31B_40P: now also RN5.6 (R3.2); no longer RN5.8 (R1.2)
- net L5_IOT63A: now also RN6.5 (R4.2); no longer RN6.7 (R2.2)
- net L9_IOT31A_40P: now also RN5.7 (R2.2)
Other:
- moved on the sheet: J3, J4

Commit message: WIP
Connections:
- net J4_IOR22A_40P is gone; now on net FT601_SIWU: J4.14 (Pin_14)
- net J7_IOT21B_40P: now also RN8.8 (R1.2)
- net K10_IOT15B_40P: now also RN9.8 (R1.2)
- net K11_IOT11A: now also RN1.5 (R4.2)
- net K1_IOR20A_40P: now also R44.2
- net K2_IOR20B_40P: now also R45.2
- net K6_IOT23B_USB_N: now also RN8.6 (R3.2)
- net K7_IOT21A_40P: now also RN8.7 (R2.2)
- net L10_IOT15A_40P: now also RN9.7 (R2.2)
- net L11_IOT11B: now also RN1.6 (R3.2)
- net L1_IOR18B_40P: now also RN1.8 (R1.2)
- net L2_IOR18A_40P: now also RN1.7 (R2.2)
- net L6_IOT23A_USB_P: now also RN8.5 (R4.2)
- net L7_IOT19A_40P: now also RN9.5 (R4.2)
- net L8_IOT19B_40P: now also RN9.6 (R3.2)
Other:
- moved on the sheet: R43, R44, R45, R46, R47, RN1, RN2, RN3, RN4, RN5, RN6, RN7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
